Commit message: ajout du cad de la main de robotiq

File: ur_description/urdf/ur5.urdf.xacro (robot description, xacro)
@@ -258,8 +258,8 @@
       <visual>
         <geometry>
-          <mesh filename="package://ur_description/meshes/ur5/visual/wrist3.dae" />
-        </geometry>
-        <material name="LightGrey">
-          <color rgba="0.7 0.7 0.7 1.0"/>
+          <mesh filename="package://ur_description/meshes/robotiq_hand/test_1.stl" />
+        </geometry>
+        <material name="LightGrey">
+          <color rgba="0.2 0.2 0.2 1.0"/>
         </material>
       </visual>
